File: schematics/schematics.kicad_sch (KiCad schematic)
At the start: 11 parts, among them Q1 SFH309, SW1 SW_Push, U1 ATtiny85-20P

Commit message: changes
Parts:
- removed Q1: SFH309, LED_THT:LED_D3.0mm_Clear, symbol Sensor_Optical:SFH309
- removed R1, R2: 1K, symbol Device:R
- removed SW1: SW_Push, Button_Switch_SMD:SW_MEC_5GSH9, symbol Switch:SW_Push
- removed U1: ATtiny85-20P, Package_DIP:DIP-8_W7.62mm, symbol MCU_Microchip_ATtiny:ATtiny85-20P
- added BT1: Battery, Battery:BatteryHolder_Keystone_2479_3xAAA, symbol Device:Battery
- added J1: Conn_01x06_Pin, Connector_PinHeader_2.54mm:PinHeader_1x06_P2.54mm_Vertical, symbol Connector:Conn_01x06_Pin
- added Q1, Q2: BC547, Package_TO_SOT_THT:TO-92_Inline, symbol Transistor_BJT:BC547
- added Q3: SFH309, LED_THT:LED_D3.0mm_Horizontal_O1.27mm_Z2.0mm, symbol Sensor_Optical:SFH309
- added R_C1: 1k, Resistor_THT:R_Axial_DIN0207_L6.3mm_D2.5mm_P10.16mm_Horizontal, symbol Device:R
- added SW1: SW_DPDT_x2, Button_Switch_SMD:SW_DPDT_CK_JS202011JCQN, symbol Switch:SW_DPDT_x2
- added U1: ATtiny414-SS, Package_SO:SOIC-14_3.9x8.7mm_P1.27mm, symbol MCU_Microchip_ATtiny:ATtiny414-SS
- C1: footprint (none) -> Capacitor_THT:CP_Radial_D5.0mm_P2.00mm
- D1, D2: footprint (none) -> LED_THT:LED_D3.0mm_Horizontal_O1.27mm_Z2.0mm
- R3, R4: value 1K -> 1k; footprint (none) -> Resistor_SMD:R_0603_1608Metric_Pad0.98x0.95mm_HandSolder
- R5: value 1K -> 4.7k; footprint (none) -> Resistor_SMD:R_0603_1608Metric_Pad0.98x0.95mm_HandSolder
Connections:
- net GND: now reaches C1.2
- net GND: now also D1.1 (K), D2.1 (K), BT1.2 (-), J1.1 (Pin_1), Q2.3 (E), U1.14 (GND)
- net at R4.2: now also U1.9 (PB0); no longer D1.1 (K)
- net at D1.2 (A): now also R4.1
- net at R3.2: now also U1.8 (PB1); no longer D2.1 (K)
- net at D2.2 (A): now also R3.1
- net at R5.2: now also SW1.1 (A), U1.10 (~{RESET}/PA0)
- new net: J1.5 (Pin_5), SW1.2 (B)
- new net: SW1.3 (C), U1.7 (PB2)
- new net: Q3.2 (E), U1.13 (PA3)
- new net: C1.1, Q2.1 (C), R_C1.1, U1.2 (PA4)
- new net: Q2.2 (B), U1.3 (PA5)
- new net: Q1.1 (C), U1.4 (PA6)
- new net: Q1.2 (B), U1.5 (PA7)
- new net: SW1.6 (C), U1.6 (PB3)
- new net: R5.1, SW1.4 (A)
- new net: J1.4 (Pin_4), SW1.5 (B)
- new net: Q1.3 (E), R_C1.2
- new net VCC: BT1.1 (+), J1.3 (Pin_3), Q3.1 (C), U1.1 (VCC)
- no-connect marks 0 -> 4

Commit message: PCB ordered
Parts:
- removed Q1, Q2: BC547, Package_TO_SOT_THT:TO-92_Inline, symbol Transistor_BJT:BC547
- added C2, C4: 0.1uF, Capacitor_SMD:C_0805_2012Metric_Pad1.18x1.45mm_HandSolder, symbol Device:C
- added Q1, Q4: MMBT3904, Package_TO_SOT_SMD:SOT-23, symbol Transistor_BJT:MMBT3904
- added U2: APE8865NR-33-HF-3, Package_TO_SOT_SMD:SOT-23, symbol Regulator_Linear:APE8865NR-33-HF-3
- BT1: footprint Battery:BatteryHolder_Keystone_2479_3xAAA -> Battery:BatteryHolder_MPD_BH-18650-PC2
- R_C1: footprint Resistor_THT:R_Axial_DIN0207_L6.3mm_D2.5mm_P10.16mm_Horizontal -> Resistor_THT:R_Axial_DIN0207_L6.3mm_D2.5mm_P2.54mm_Vertical
Connections:
- net GND: now also C2.2, C4.2, Q1.2 (E), U2.3 (GND)
- net VCC: now also C4.1, U2.1 (VI); no longer BT1.1 (+), J1.3 (Pin_3)
- net at C1.1, R_C1.1, U1.2 (PA4): now also Q1.3 (C)
- net at U1.3 (PA5): now also Q1.1 (B)
- net at U1.4 (PA6): now also Q4.3 (C)
- net at U1.5 (PA7): now also Q4.1 (B)
- net at R_C1.2: now also Q4.2 (E)
- new net: BT1.1 (+), C2.1, J1.3 (Pin_3), U2.2 (VO)
Other:
- moved on the sheet: BT1, J1
