File: schematics/schematics.kicad_pcb (KiCad board)
At the start: 2 copper layers, 14 parts, among them J1 Conn_01x06_Pin, Q1 BC547, Q2 BC547, Q3 SFH309, SW1 SW_DPDT_x2, U1 ATtiny414-SS

Commit message: pcb
Parts:
- Q1, Q2: footprint Package_TO_SOT_THT:TO-92_Inline -> Package_TO_SOT_SMD:SOT-23-3
- R_C1: footprint Resistor_THT:R_Axial_DIN0207_L6.3mm_D2.5mm_P10.16mm_Horizontal -> Resistor_THT:R_Axial_DIN0207_L6.3mm_D2.5mm_P2.54mm_Vertical
- moved R_C1 33.0 mm to (106.7, 143.3), turned to 90 degrees
- moved Q2 26.7 mm to (99.6, 147.6), turned to 180 degrees
- moved C1 20.1 mm to (105.7, 151.4), turned to 0 degrees
- moved Q1 6.27 mm to (99.6, 142.5), turned to 180 degrees
Routing:
- net Net-(Q2-C): track 0.00 -> 20.9 mm
- net Net-(Q1-E): track 0.00 -> 8.99 mm
- net Net-(Q2-B): track 0.00 -> 6.28 mm
- net Net-(Q1-B): track 0.00 -> 5.81 mm
- net Net-(Q1-C): track 0.00 -> 5.55 mm

Commit message: PCB ordered
Parts:
- removed Q2: BC547, Package_TO_SOT_SMD:SOT-23-3
- added C2: 0.1uF, Capacitor_SMD:C_0805_2012Metric_Pad1.18x1.45mm_HandSolder, F.Cu at (109.3, 155.3)
- added C4: 0.1uF, Capacitor_SMD:C_0805_2012Metric_Pad1.18x1.45mm_HandSolder, F.Cu at (82.5, 157.2)
- added Q4: MMBT3904, Package_TO_SOT_SMD:SOT-23, F.Cu at (100.2, 141.5)
- added Q5: APE8865NR-33-HF-3, Package_TO_SOT_SMD:SOT-23, F.Cu at (108.3, 150.9)
- BT1: footprint Battery:BatteryHolder_Keystone_2479_3xAAA -> Battery:BatteryHolder_MPD_BH-18650-PC2
- Q1: value BC547 -> MMBT3904; footprint Package_TO_SOT_SMD:SOT-23-3 -> Package_TO_SOT_SMD:SOT-23
- moved BT1 12.9 mm to (114.3, 149.5)
- moved R4 5.09 mm to (81.5, 141.0)
- moved C1 4.51 mm to (101.3, 152.1)
- moved R3 4.17 mm to (85.4, 139.7)
- moved Q1 3.23 mm to (100.2, 145.7), turned to 0 degrees
- moved D1 2.81 mm to (76.2, 146.3)
- moved D2 2.81 mm to (76.2, 140.0)
- moved R_C1 2.05 mm to (105.7, 145.0)
- moved J1 1.52 mm to (88.9, 158.5)
- moved R5 0.91 mm to (85.4, 142.2)
Connections:
- BT1 pad 1: VCC -> Net-(BT1-+)
- C1 pad 1: Net-(Q2-C) -> Net-(Q1-C)
- J1 pad 3: VCC -> Net-(BT1-+)
- Q1 pad 1: Net-(Q1-C) -> Net-(Q1-B)
- Q1 pad 2: Net-(Q1-B) -> GND
- Q1 pad 3: Net-(Q1-E) -> Net-(Q1-C)
- R_C1 pad 1: Net-(Q2-C) -> Net-(Q1-C)
- R_C1 pad 2: Net-(Q1-E) -> Net-(Q4-E)
- U1 pad 2: Net-(Q2-C) -> Net-(Q1-C)
- U1 pad 3: Net-(Q2-B) -> Net-(Q1-B)
- U1 pad 4: Net-(Q1-C) -> Net-(Q4-C)
- U1 pad 5: Net-(Q1-B) -> Net-(Q4-B)
Routing:
- net Net-(Q1-C): track 5.55 -> 610.5 mm
- net VCC: track 0.00 -> 44.4 mm, vias 0 -> 2
- net Net-(BT1-+): track 0.00 -> 26.7 mm
- net Net-(Q3-E): track 0.00 -> 25.2 mm, vias 0 -> 1
- net Net-(Q2-C): track 20.9 -> 0.00 mm
- net Net-(Q1-E): track 8.99 -> 0.00 mm
- net Net-(D1-A): track 4.17 -> 11.3 mm
- net Net-(Q4-C): track 0.00 -> 6.84 mm
- net Net-(Q4-E): track 0.00 -> 6.47 mm
- net Net-(Q2-B): track 6.28 -> 0.00 mm
- net Net-(U1-PB0): track 13.8 -> 7.79 mm
- net GND: track 0.00 -> 5.94 mm, vias 0 -> 4
- net Net-(D2-A): track 4.17 -> 9.86 mm
- net Net-(U1-PB1): track 9.31 -> 3.88 mm
- net Net-(Q4-B): track 0.00 -> 4.74 mm
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- added copper zone on F.Cu, net GND
Other:
- board outline added: 640.5 x 25 mm
- board text added: "SSCS-Arduino-Contest 2024 Submission Kellen Yu Cost-effective soil moisture sensor array"

Commit message: working on interrupts
Routing:
- net Net-(Q1-C): track 610.5 -> 507.4 mm
Other:
- board size 640.5 x 25 mm -> 541 x 25 mm
Changed lines of the file:
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@@
 	)
 	(gr_line
-		(start 74 137)
-		(end 700 137)
+		(start 598.5 162)
+		(end 615 149.5)
 		(stroke
 			(width 0.05)
@@
 	)
 	(gr_line
-		(start 714.5 150)
-		(end 700 162)
+		(start 74 137)
+		(end 598.5 137)
+		(stroke
+			(width 0.05)
+			(type default)
+		)
+		(layer "Edge.Cuts")
+	)
+	(gr_line
+		(start 615 149.5)
+		(end 598.5 137)
 		(stroke
 			(width 0.05)
@@
 		(layer "Edge.Cuts")
 	)
-	(gr_line
-		(start 700 137)
-		(end 714.5 150)
-		(stroke
-			(width 0.05)
-			(type default)
-		)
-		(layer "Edge.Cuts")
-	)
 	(gr_circle
 		(center 81.5 152)
@@
 	)
 	(gr_line
-		(start 700 162)
+		(start 598.5 162)
 		(end 74 162)
 		(stroke
@@
 		(layer "Dwgs.User")
 		(pts
-			(xy 195 142) (xy 195 137)
+			(xy 195 142.5) (xy 195 137.5)
 		)
 		(height 6)
 		(gr_text "5.0000 mm"
-			(at 199.85 139.5 90)
+			(at 199.85 140 90)
 			(layer "Dwgs.User")
 			(effects
@@
 			(extension_offset 0.5) keep_text_aligned)
 	)
+	(dimension
+		(type aligned)
+		(layer "Dwgs.User")
+		(pts
+			(xy 615.25 149.5) (xy 615.25 137)
+		)
+		(height 3.25)
+		(gr_text "12.5000 mm"
+			(at 617.35 143.25 90)
+			(layer "Dwgs.User")
+			(effects
+				(font
+					(size 1 1)
+					(thickness 0.15)
+				)
+			)
+		)
+		(format
+			(prefix "")
+			(suffix "")
+			(units 3)
+			(units_format 1)
+			(precision 4)
+		)
+		(style
+			(thickness 0.1)
+			(arrow_length 1.27)
+			(text_position_mode 0)
+			(extension_height 0.58642)
+			(extension_offset 0.5) keep_text_aligned)
+	)
+	(dimension
+		(type aligned)
+		(layer "Dwgs.User")
+		(pts
+			(xy 615 149.5) (xy 615 162)
+		)
+		(height -3.5)
+		(gr_text "12.5000 mm"
+			(at 617.35 155.75 90)
+			(layer "Dwgs.User")
+			(effects
+				(font
+					(size 1 1)
+					(thickness 0.15)
+				)
+			)
+		)
+		(format
+			(prefix "")
+			(suffix "")
+			(units 3)
+			(units_format 1)
+			(precision 4)
+		)
+		(style
+			(thickness 0.1)
+			(arrow_length 1.27)
+			(text_position_mode 0)
+			(extension_height 0.58642)
+			(extension_offset 0.5) keep_text_aligned)
+	)
+	(dimension
+		(type aligned)
+		(layer "Dwgs.User")
+		(pts
+			(xy 111.3 159.55) (xy 189.3 159.55)
+		)
+		(height 6.565999)
+		(gr_text "78.0000 mm"
+			(at 150.3 164.965999 0)
+			(layer "Dwgs.User")
+			(effects
+				(font
+					(size 1 1)
+					(thickness 0.15)
+				)
+			)
+		)
+		(format
+			(prefix "")
+			(suffix "")
+			(units 3)
+			(units_format 1)
+			(precision 4)
+		)
+		(style
+			(thickness 0.1)
+			(arrow_length 1.27)
+			(text_position_mode 0)
+			(extension_height 0.58642)
+			(extension_offset 0.5) keep_text_aligned)
+	)
+	(dimension
+		(type aligned)
+		(layer "Dwgs.User")
+		(pts
+			(xy 114.3 149.5) (xy 186.309 149.479)
+		)
+		(height 24.374097)
+		(gr_text "72.0090 mm"
+			(at 150.311273 172.713596 0.0167091799)
+			(layer "Dwgs.User")
+			(effects
+				(font
+					(size 1 1)
+					(thickness 0.15)
+				)
+			)
+		)
+		(format
+			(prefix "")
+			(suffix "")
+			(units 3)
+			(units_format 1)
+			(precision 4)
+		)
+		(style
+			(thickness 0.1)
+			(arrow_length 1.27)
+			(text_position_mode 0)
+			(extension_height 0.58642)
+			(extension_offset 0.5) keep_text_aligned)
+	)
 	(via
 		(at 106.7785 158.7785)
@@
 	)
 	(segment
+		(start 105.664 145.034)
+		(end 105.664 147.32)
+		(width 0.2)
+		(layer "F.Cu")
+		(net 10)
+	)
+	(segment
 		(start 101.279888 152.146)
 		(end 100.076 152.146)
@@
 	)
 	(segment
-		(start 210 150)
-		(end 206.75 146.75)
-		(width 0.2)
+		(start 212.5 149.5)
+		(end 590.5 149.5)
+		(width 14)
 		(layer "F.Cu")
 		(net 10)
@@
 	)
 	(segment
-		(start 105.664 145.034)
-		(end 105.664 147.761888)
-		(width 0.2)
-		(layer "F.Cu")
-		(net 10)
-	)
-	(segment
 		(start 96.774 148.844)
 		(end 96.774 146.664001)
@@
 	)
 	(segment
+		(start 105.664 147.32)
+		(end 105.664 147.761888)
+		(width 0.2)
+		(layer "F.Cu")
+		(net 10)
+	)
+	(segment
 		(start 96.774 146.664001)
 		(end 96.159999 146.05)
@@
 	)
 	(segment
-		(start 210 150)
-		(end 690.5 150)
-		(width 14)
+		(start 105.734 147.25)
+		(end 105.664 147.32)
+		(width 0.2)
 		(layer "F.Cu")
 		(net 10)
@@
 	)
 	(segment
+		(start 210 150.5)
+		(end 206.75 147.25)
+		(width 0.2)
+		(layer "F.Cu")
+		(net 10)
+	)
+	(segment
+		(start 206.75 147.25)
+		(end 105.734 147.25)
+		(width 0.2)
+		(layer "F.Cu")
+		(net 10)
+	)
+	(segment
 		(start 103.632 145.669)
 		(end 104.267 145.034)
-		(width 0.2)
-		(layer "F.Cu")
-		(net 10)
-	)
-	(segment
-		(start 106.675888 146.75)
-		(end 105.503944 147.921944)
-		(width 0.2)
-		(layer "F.Cu")
-		(net 10)
-	)
-	(segment
-		(start 206.75 146.75)
-		(end 106.675888 146.75)
 		(width 0.2)
 		(layer "F.Cu")
@@
 		(polygon
 			(pts
-				(xy 74 162) (xy 74 137) (xy 715.5 137) (xy 715.5 162)
+				(xy 74 162) (xy 74 137) (xy 615.779 137) (xy 615.779 162)
 			)
 		)
